File: Hardware/PCB/pcb_telemetria_caqui.sch (EAGLE design)
At the start: 35 parts

Commit message: att
Parts:
- removed TBEAM_LEFT, TBEAM_RIGHT: 61301311121, Headers:61301311121
- added U$1: TTGOBEAM, bibliotecattgo:TTGOBEAM
Connections:
- new net GND1: U$1.GND1
- new net GND2: U$1.GND2
- net 0: now also U$1.0; no longer TBEAM_RIGHT.5
- net 13: now also U$1.13; no longer TBEAM_LEFT.4
- net 14: now also U$1.14; no longer TBEAM_LEFT.5
- net 2: now also U$1.2; no longer TBEAM_LEFT.3
- net 21: now also U$1.21; no longer TBEAM_RIGHT.10
- net 22: now also U$1.22; no longer TBEAM_RIGHT.9
- net 23: now also U$1.23; no longer TBEAM_RIGHT.3
- net 25: now also U$1.25; no longer TBEAM_LEFT.6
- net 3.3V: now also U$1.3.3V; no longer TBEAM_RIGHT.11
- net 32: now also U$1.32; no longer TBEAM_LEFT.8
- net 33: now also U$1.33; no longer TBEAM_LEFT.7
- net 34: now also U$1.34; no longer TBEAM_LEFT.10
- net 35: now also U$1.35; no longer TBEAM_LEFT.9
- net 3V3: now also U$1.3V3; no longer TBEAM_RIGHT.7
- net 4: now also U$1.4; no longer TBEAM_RIGHT.4
- net 5V: now also U$1.5V; no longer TBEAM_LEFT.1
- net C0: now also R10.2, R9.1; no longer R3.2, R4.1
- net C1: now also R7.2, R8.1; no longer R5.1, R6.2
- net C2: now also R5.1, R6.2; no longer R7.2, R8.1
- net C3: now also R3.2, R4.1; no longer R10.2, R9.1
- net GND: now also U$1.GND; no longer TBEAM_LEFT.2, TBEAM_RIGHT.6, TBEAM_RIGHT.8
- net LORA1: now also U$1.LORA1; no longer TBEAM_RIGHT.13
- net LORA2: now also U$1.LORA2; no longer TBEAM_RIGHT.12
- net RST: now also U$1.RST; no longer TBEAM_LEFT.11
- net RX: now also U$1.RX; no longer TBEAM_RIGHT.2
- net TX: now also U$1.TX; no longer TBEAM_RIGHT.1
- net VN: now also U$1.VN; no longer TBEAM_LEFT.12
- net VP: now also U$1.VP; no longer TBEAM_LEFT.13

Commit message: uplix
Parts:
- removed BB_BE_C: CURRENT-SENSOR-ACS712, diy-modules:CURRENT-SENSOR-ACS712
- added C_BP: CURRENT-SENSOR-ACS712, diy-modules:CURRENT-SENSOR-ACS712
- added R25, R27: 2.2k, rcl:R-EU_0204/7
- added R26, R28: 3.9k, rcl:R-EU_0204/7
- added TEMP: (no value), con-amp-quick:M02
Connections:
- removed net EN: HC4067.EN
- removed net S0: HC4067.S0
- removed net S1: HC4067.S1
- removed net S2: HC4067.S2
- removed net S3: HC4067.S3
- removed net SIG: HC4067.SIG
- removed net VCC: C_BAUX.VCC, HC4067.VCC
- new net N$1: C_BP.OUT, R25.2
- new net N$2: C_BAUX.OUT, R27.2
- net 0: now also HC4067.S3
- net 13: now also R1.1, R2.2; no longer R23.2, R24.1
- net 14: now also R21.1, R22.2; no longer R13.1, R14.2
- net 2: now also R13.1, R14.2; no longer R11.2, R12.1
- net 21: now also SHUNTS.1; no longer SHUNTS.2
- net 22: now also SHUNTS.2; no longer SHUNTS.1
- net 23: now also HC4067.EN
- net 25: now also R11.2, R12.1; no longer R1.1, R2.2
- net 32: now also HC4067.S0
- net 33: now also R27.1, R28.1; no longer C_BAUX.OUT
- net 34: now also HC4067.S2
- net 35: now also HC4067.S1
- net 4: now also HC4067.SIG
- net 5V: now also C_BAUX.VCC, C_BP.VCC, HC4067.VCC
- net BAT_AUX: now also R21.2, SL3.1; no longer R23.1, SL4.3
- net C10: now also TEMP.1
- net C4: now also R23.2, R24.1; no longer R21.1, R22.2
- net C5: now also R15.2, R16.1; no longer R19.2, R20.1
- net C7: now also R19.2, R20.1; no longer R15.2, R16.1
- net C8: now also R25.1, R26.1
- net C9: now also TEMP.2
- net COOLER_E: now also R23.1, SL4.3; no longer R21.2, SL3.1
- net GND: now also C_BP.GND, R26.2, R28.2
Other:
- moved on the sheet: C_BAUX, HC4067, R1, R11, R12, R13, R14, R15, R16, R17, R18, R19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

Commit message: up
Parts:
- added IC1: 7805TV, linear:7805TV
- added SUPPLY: (no value), con-amp-quick:M02
Connections:
- new net VI: IC1.VI, SUPPLY.2
- new net VO: IC1.VO
- net 3V3: now also HC4067.VCC
- net 5V: no longer HC4067.VCC
- net GND: now also IC1.GND, SUPPLY.1
Changed lines of the file:
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@@
 <?xml version="1.0" encoding="utf-8"?>
 <!DOCTYPE eagle SYSTEM "eagle.dtd">
-<eagle version="9.4.2">
+<eagle version="9.5.0">
 <drawing>
 <settings>
@@
 <part name="GND8" library="supply1" library_urn="urn:adsk.eagle:library:371" deviceset="GND" device=""/>
 <part name="TEMP" library="con-amp-quick" library_urn="urn:adsk.eagle:library:125" deviceset="M02" device="" package3d_urn="urn:adsk.eagle:package:5956/1"/>
+<part name="IC1" library="linear" library_urn="urn:adsk.eagle:library:262" deviceset="78*" device="TV" package3d_urn="urn:adsk.eagle:package:16417/2" technology="05"/>
+<part name="SUPPLY" library="con-amp-quick" library_urn="urn:adsk.eagle:library:125" deviceset="M02" device="" package3d_urn="urn:adsk.eagle:package:5956/1"/>
 </parts>
 <sheets>
@@
 <attribute name="NAME" x="-76.962" y="-58.928" size="1.778" layer="95"/>
 </instance>
+<instance part="IC1" gate="A1" x="-157.48" y="88.9" smashed="yes">
+<attribute name="NAME" x="-165.1" y="94.615" size="1.778" layer="95"/>
+<attribute name="VALUE" x="-165.1" y="92.075" size="1.778" layer="96"/>
+</instance>
+<instance part="SUPPLY" gate="G$1" x="-156.21" y="46.99" smashed="yes" rot="R90">
+<attribute name="VALUE" x="-151.13" y="44.45" size="1.778" layer="96" rot="R90"/>
+<attribute name="NAME" x="-161.798" y="46.228" size="1.778" layer="95" rot="R180"/>
+</instance>
 </instances>
 <busses>
@@
 <wire x1="-120.396" y1="93.98" x2="-120.396" y2="97.282" width="0.1524" layer="91"/>
 </segment>
+<segment>
+<wire x1="-156.21" y1="54.61" x2="-156.21" y2="66.04" width="0.1524" layer="91"/>
+<pinref part="SUPPLY" gate="G$1" pin="1"/>
+<label x="-154.94" y="66.04" size="1.778" layer="95" rot="R270"/>
+</segment>
+<segment>
+<pinref part="IC1" gate="A1" pin="GND"/>
+<wire x1="-157.48" y1="81.28" x2="-157.48" y2="68.58" width="0.1524" layer="91"/>
+<label x="-157.48" y="71.12" size="1.778" layer="95" rot="R90"/>
+</segment>
 </net>
 <net name="22" class="0">
@@
 </segment>
 <segment>
-<pinref part="HC4067" gate="G$1" pin="VCC"/>
-<wire x1="42.672" y1="150.622" x2="42.672" y2="160.782" width="0.1524" layer="91"/>
-<label x="42.672" y="160.782" size="1.778" layer="95" rot="R90" align="bottom-right"/>
-</segment>
-<segment>
-<pinref part="C_BP" gate="G$1" pin="VCC"/>
-<wire x1="-141.986" y1="144.526" x2="-132.842" y2="144.526" width="0.1524" layer="91"/>
-<label x="-132.588" y="144.78" size="1.778" layer="95" align="bottom-right"/>
-</segment>
-<segment>
 <pinref part="C_BAUX" gate="G$1" pin="VCC"/>
 <wire x1="-140.208" y1="112.522" x2="-130.556" y2="112.522" width="0.1524" layer="91"/>
 <label x="-133.604" y="112.776" size="1.778" layer="95"/>
 </segment>
+<segment>
+<pinref part="C_BP" gate="G$1" pin="VCC"/>
+<wire x1="-141.986" y1="144.526" x2="-133.096" y2="144.526" width="0.1524" layer="91"/>
+<label x="-133.858" y="146.05" size="1.778" layer="95"/>
+</segment>
 </net>
 <net name="TX" class="0">
@@
 <wire x1="-7.112" y1="127.762" x2="5.588" y2="127.762" width="0.1524" layer="91"/>
 <label x="6.096" y="128.016" size="1.778" layer="95" align="bottom-right"/>
+</segment>
+<segment>
+<pinref part="HC4067" gate="G$1" pin="VCC"/>
+<wire x1="42.672" y1="150.622" x2="42.672" y2="160.782" width="0.1524" layer="91"/>
+<label x="42.418" y="156.718" size="1.778" layer="95" rot="R90"/>
 </segment>
 </net>
@@
 </segment>
 </net>
+<net name="VI" class="0">
+<segment>
+<pinref part="SUPPLY" gate="G$1" pin="2"/>
+<wire x1="-158.75" y1="54.61" x2="-158.75" y2="66.04" width="0.1524" layer="91"/>
+<label x="-160.02" y="66.04" size="1.778" layer="95" rot="R90"/>
+</segment>
+<segment>
+<pinref part="IC1" gate="A1" pin="VI"/>
+<wire x1="-167.64" y1="88.9" x2="-180.34" y2="88.9" width="0.1524" layer="91"/>
+<label x="-177.8" y="88.9" size="1.778" layer="95"/>
+</segment>
+</net>
+<net name="VO" class="0">
+<segment>
+<pinref part="IC1" gate="A1" pin="VO"/>
+<wire x1="-147.32" y1="88.9" x2="-134.62" y2="88.9" width="0.1524" layer="91"/>
+<label x="-137.16" y="91.44" size="1.778" layer="95"/>
+</segment>
+</net>

Commit message: Changes in the board and code
mudancas no codigo e placa
Parts:
- added U$2: DC-DC-STEP-DOWN-LM2596, diy-modules:DC-DC-STEP-DOWN-LM2596
Changed lines of the file:
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@@
 <?xml version="1.0" encoding="utf-8"?>
 <!DOCTYPE eagle SYSTEM "eagle.dtd">
-<eagle version="9.5.0">
+<eagle version="9.4.2">
 <drawing>
 <settings>
@@
 <part name="IC1" library="linear" library_urn="urn:adsk.eagle:library:262" deviceset="78*" device="TV" package3d_urn="urn:adsk.eagle:package:16417/2" technology="05"/>
 <part name="SUPPLY" library="con-amp-quick" library_urn="urn:adsk.eagle:library:125" deviceset="M02" device="" package3d_urn="urn:adsk.eagle:package:5956/1"/>
+<part name="U$2" library="diy-modules" deviceset="DC-DC-STEP-DOWN-LM2596" device=""/>
 </parts>
 <sheets>
@@
 <attribute name="NAME" x="-161.798" y="46.228" size="1.778" layer="95" rot="R180"/>
 </instance>
+<instance part="U$2" gate="G$1" x="-5.08" y="182.88" smashed="yes">
+<attribute name="NAME" x="-17.78" y="198.12" size="1.778" layer="95"/>
+<attribute name="VALUE" x="-17.78" y="195.58" size="1.778" layer="96"/>
+</instance>
 </instances>

Commit message: ultima att
up
Parts:
- removed U$2: DC-DC-STEP-DOWN-LM2596, diy-modules:DC-DC-STEP-DOWN-LM2596
- added TEMP2: (no value), con-amp-quick:M02
- renumbered TEMP to TEMP1
Connections:
- new net C21: TEMP1.2, TEMP2.2
- new net C22: TEMP1.1, TEMP2.1
- net 13: no longer R1.1, R2.2
- net 14: no longer R21.1, R22.2
- net 2: no longer R13.1, R14.2
- net 25: no longer R11.2, R12.1
- net 33: no longer R27.1, R28.1
- net C10: now also R1.1, R2.2; no longer TEMP1.1
- net C11: now also R11.2, R12.1
- net C12: now also R21.1, R22.2
- net C13: now also R13.1, R14.2
- net C9: now also R27.1, R28.1; no longer TEMP1.2
Changed lines of the file:
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@@
 <part name="R28" library="rcl" library_urn="urn:adsk.eagle:library:334" deviceset="R-EU_" device="0204/7" package3d_urn="urn:adsk.eagle:package:23498/2" value="3.9k"/>
 <part name="GND8" library="supply1" library_urn="urn:adsk.eagle:library:371" deviceset="GND" device=""/>
-<part name="TEMP" library="con-amp-quick" library_urn="urn:adsk.eagle:library:125" deviceset="M02" device="" package3d_urn="urn:adsk.eagle:package:5956/1"/>
+<part name="TEMP1" library="con-amp-quick" library_urn="urn:adsk.eagle:library:125" deviceset="M02" device="" package3d_urn="urn:adsk.eagle:package:5956/1"/>
 <part name="IC1" library="linear" library_urn="urn:adsk.eagle:library:262" deviceset="78*" device="TV" package3d_urn="urn:adsk.eagle:package:16417/2" technology="05"/>
 <part name="SUPPLY" library="con-amp-quick" library_urn="urn:adsk.eagle:library:125" deviceset="M02" device="" package3d_urn="urn:adsk.eagle:package:5956/1"/>
-<part name="U$2" library="diy-modules" deviceset="DC-DC-STEP-DOWN-LM2596" device=""/>
+<part name="TEMP2" library="con-amp-quick" library_urn="urn:adsk.eagle:library:125" deviceset="M02" device="" package3d_urn="urn:adsk.eagle:package:5956/1"/>
 </parts>
 <sheets>
@@
 <attribute name="VALUE" x="-122.936" y="88.9" size="1.778" layer="96"/>
 </instance>
-<instance part="TEMP" gate="G$1" x="-82.55" y="-59.69" smashed="yes" rot="R270">
+<instance part="TEMP1" gate="G$1" x="-82.55" y="-59.69" smashed="yes" rot="R270">
 <attribute name="VALUE" x="-87.63" y="-57.15" size="1.778" layer="96" rot="R270"/>
 <attribute name="NAME" x="-76.962" y="-58.928" size="1.778" layer="95"/>
@@
 <attribute name="NAME" x="-161.798" y="46.228" size="1.778" layer="95" rot="R180"/>
 </instance>
-<instance part="U$2" gate="G$1" x="-5.08" y="182.88" smashed="yes">
-<attribute name="NAME" x="-17.78" y="198.12" size="1.778" layer="95"/>
-<attribute name="VALUE" x="-17.78" y="195.58" size="1.778" layer="96"/>
+<instance part="TEMP2" gate="G$1" x="-64.77" y="-59.69" smashed="yes" rot="R270">
+<attribute name="VALUE" x="-69.85" y="-57.15" size="1.778" layer="96" rot="R270"/>
+<attribute name="NAME" x="-59.182" y="-58.928" size="1.778" layer="95"/>
 </instance>
 </instances>
@@
 <label x="-50.292" y="117.602" size="1.778" layer="95"/>
 </segment>
-<segment>
-<pinref part="R14" gate="G$1" pin="2"/>
-<pinref part="R13" gate="G$1" pin="1"/>
-<wire x1="-137.668" y1="-10.16" x2="-137.668" y2="-7.62" width="0.1524" layer="91"/>
-<wire x1="-137.668" y1="-7.62" x2="-144.78" y2="-7.62" width="0.1524" layer="91"/>
-<junction x="-137.668" y="-7.62"/>
-<label x="-144.78" y="-5.08" size="1.778" layer="95"/>
-</segment>
 </net>
 <net name="33" class="0">
@@
 <label x="-50.292" y="127.762" size="1.778" layer="95"/>
 </segment>
-<segment>
-<pinref part="R27" gate="G$1" pin="1"/>
-<pinref part="R28" gate="G$1" pin="1"/>
-<wire x1="-120.396" y1="107.442" x2="-120.396" y2="109.982" width="0.1524" layer="91"/>
-<wire x1="-120.396" y1="109.982" x2="-116.84" y2="109.982" width="0.1524" layer="91"/>
-<junction x="-120.396" y="109.982"/>
-<label x="-116.84" y="111.76" size="1.778" layer="95"/>
-</segment>
 </net>
 <net name="25" class="0">
@@
 <label x="-50.292" y="125.222" size="1.778" layer="95"/>
 </segment>
-<segment>
-<pinref part="R12" gate="G$1" pin="1"/>
-<pinref part="R11" gate="G$1" pin="2"/>
-<wire x1="3.81" y1="-12.7" x2="3.81" y2="-10.16" width="0.1524" layer="91"/>
-<wire x1="3.81" y1="-10.16" x2="-1.27" y2="-10.16" width="0.1524" layer="91"/>
-<junction x="3.81" y="-10.16"/>
-</segment>
 </net>
 <net name="14" class="0">
@@
 <label x="-50.292" y="122.682" size="1.778" layer="95"/>
 </segment>
-<segment>
-<pinref part="R22" gate="G$1" pin="2"/>
-<pinref part="R21" gate="G$1" pin="1"/>
-<wire x1="64.262" y1="66.802" x2="64.262" y2="69.342" width="0.1524" layer="91"/>
-<wire x1="64.262" y1="69.342" x2="58.42" y2="69.342" width="0.1524" layer="91"/>
-<junction x="64.262" y="69.342"/>
-</segment>
 </net>
 <net name="13" class="0">
@@
 <wire x1="-40.132" y1="120.142" x2="-50.292" y2="120.142" width="0.1524" layer="91"/>
 <label x="-50.292" y="120.142" size="1.778" layer="95"/>
-</segment>
-<segment>
-<pinref part="R2" gate="G$1" pin="2"/>
-<pinref part="R1" gate="G$1" pin="1"/>
-<wire x1="-63.5" y1="-10.16" x2="-63.5" y2="-7.62" width="0.1524" layer="91"/>
-<wire x1="-63.5" y1="-7.62" x2="-71.12" y2="-7.62" width="0.1524" layer="91"/>
-<junction x="-63.5" y="-7.62"/>
-<label x="-71.12" y="-5.08" size="1.778" layer="95"/>
 </segment>
 </net>
@@
 <label x="22.352" y="112.522" size="1.778" layer="95" rot="R90"/>
 </segment>
+<segment>
+<pinref part="R14" gate="G$1" pin="2"/>
+<pinref part="R13" gate="G$1" pin="1"/>
+<wire x1="-137.668" y1="-10.16" x2="-137.668" y2="-7.62" width="0.1524" layer="91"/>
+<wire x1="-137.668" y1="-7.62" x2="-142.24" y2="-7.62" width="0.1524" layer="91"/>
+<junction x="-137.668" y="-7.62"/>
+<label x="-142.24" y="-5.08" size="1.778" layer="95"/>
+</segment>
 </net>
 <net name="C12" class="0">
@@
 <label x="24.892" y="112.522" size="1.778" layer="95" rot="R90"/>
 </segment>
+<segment>
+<pinref part="R22" gate="G$1" pin="2"/>
+<pinref part="R21" gate="G$1" pin="1"/>
+<wire x1="64.262" y1="66.802" x2="64.262" y2="69.342" width="0.1524" layer="91"/>
+<wire x1="64.262" y1="69.342" x2="59.436" y2="69.342" width="0.1524" layer="91"/>
+<junction x="64.262" y="69.342"/>
+<label x="59.436" y="73.66" size="1.778" layer="95"/>
+</segment>
 </net>
 <net name="C11" class="0">
@@
 <label x="27.432" y="112.522" size="1.778" layer="95" rot="R90"/>
 </segment>
+<segment>
+<pinref part="R12" gate="G$1" pin="1"/>
+<pinref part="R11" gate="G$1" pin="2"/>
+<wire x1="3.81" y1="-12.7" x2="3.81" y2="-10.16" width="0.1524" layer="91"/>
+<wire x1="3.81" y1="-10.16" x2="-2.54" y2="-10.16" width="0.1524" layer="91"/>
+<junction x="3.81" y="-10.16"/>
+<label x="-2.54" y="-7.62" size="1.778" layer="95"/>
+</segment>
 </net>
 <net name="C10" class="0">
@@
 </segment>
 <segment>
-<pinref part="TEMP" gate="G$1" pin="1"/>
-<wire x1="-82.55" y1="-67.31" x2="-82.55" y2="-72.136" width="0.1524" layer="91"/>
-<label x="-83.82" y="-73.66" size="1.778" layer="95" rot="R270"/>
+<pinref part="R2" gate="G$1" pin="2"/>
+<pinref part="R1" gate="G$1" pin="1"/>
+<wire x1="-63.5" y1="-10.16" x2="-63.5" y2="-7.62" width="0.1524" layer="91"/>
+<wire x1="-63.5" y1="-7.62" x2="-71.12" y2="-7.62" width="0.1524" layer="91"/>
+<junction x="-63.5" y="-7.62"/>
+<label x="-71.12" y="-5.08" size="1.778" layer="95"/>
 </segment>
 </net>
@@
 </segment>
 <segment>
-<pinref part="TEMP" gate="G$1" pin="2"/>
-<wire x1="-80.01" y1="-67.31" x2="-80.01" y2="-71.882" width="0.1524" layer="91"/>
-<label x="-80.264" y="-73.66" size="1.778" layer="95" rot="R270"/>
+<pinref part="R28" gate="G$1" pin="1"/>
+<pinref part="R27" gate="G$1" pin="1"/>
+<wire x1="-120.396" y1="107.442" x2="-120.396" y2="109.982" width="0.1524" layer="91"/>
+<wire x1="-120.396" y1="109.982" x2="-115.062" y2="109.982" width="0.1524" layer="91"/>
+<junction x="-120.396" y="109.982"/>
+<label x="-115.57" y="111.252" size="1.778" layer="95"/>
 </segment>
 </net>
@@
 </segment>
 </net>
+<net name="C22" class="0">
+<segment>
+<pinref part="TEMP1" gate="G$1" pin="1"/>
+<wire x1="-82.55" y1="-67.31" x2="-82.55" y2="-73.152" width="0.1524" layer="91"/>
+<label x="-88.9" y="-71.12" size="1.778" layer="95"/>
+</segment>
+<segment>
+<pinref part="TEMP2" gate="G$1" pin="1"/>
+<wire x1="-64.77" y1="-67.31" x2="-64.77" y2="-73.406" width="0.1524" layer="91"/>
+<label x="-68.58" y="-71.12" size="1.778" layer="95" rot="R270"/>
+</segment>
+</net>
+<net name="C21" class="0">
+<segment>
+<pinref part="TEMP1" gate="G$1" pin="2"/>
+<wire x1="-80.01" y1="-67.31" x2="-80.01" y2="-72.898" width="0.1524" layer="91"/>
+<label x="-78.74" y="-71.12" size="1.778" layer="95"/>
+</segment>
+<segment>
+<pinref part="TEMP2" gate="G$1" pin="2"/>
+<wire x1="-62.23" y1="-67.31" x2="-62.23" y2="-73.406" width="0.1524" layer="91"/>
+<label x="-60.96" y="-71.12" size="1.778" layer="95" rot="R270"/>
+</segment>
+</net>

Commit message: att nos pinos e adicao de regulador pwm
tired
Parts:
- removed IC1: 7805TV, linear:7805TV
- added U$2: DC-DC-STEP-DOWN-LM2596, diy-modules:DC-DC-STEP-DOWN-LM2596
Connections:
- removed net C21: TEMP1.2, TEMP2.2
- removed net C22: TEMP1.1, TEMP2.1
- removed net VO: IC1.VO
- new net VCC: U$2.OUT+
- net 21: now also TEMP1.2, TEMP2.2
- net 22: now also TEMP1.1, TEMP2.1
- net C10: now also R21.1, R22.2; no longer R1.1, R2.2
- net C11: now also R1.1, R2.2; no longer R11.2, R12.1
- net C12: now also R13.1, R14.2; no longer R21.1, R22.2
- net C13: now also R27.1, R28.1; no longer R13.1, R14.2
- net C4: now also R11.2, R12.1; no longer R23.2, R24.1
- net C5: now also R23.2, R24.1; no longer R15.2, R16.1
- net C6: now also R15.2, R16.1; no longer R17.1, R18.2
- net C7: now also R17.1, R18.2; no longer R19.2, R20.1
- net C8: now also R19.2, R20.1; no longer R25.1, R26.1
- net C9: now also R25.1, R26.1; no longer R27.1, R28.1
- net GND: now also U$2.IN-, U$2.OUT-; no longer IC1.GND
- net VI: now also U$2.IN+; no longer IC1.VI
Other:
- moved on the sheet: SUPPLY
