File: Hardware/PCB/pcb_telemetria.sch (EAGLE design)
At the start: 33 parts

Commit message: update
adicao de rotas na pcb
Connections:
- net 25: no longer C_BAUX.OUT
- net 33: now also C_BAUX.OUT
- net C5: now also R20.1
Changed lines of the file:
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@@
 <?xml version="1.0" encoding="utf-8"?>
 <!DOCTYPE eagle SYSTEM "eagle.dtd">
-<eagle version="9.5.0">
+<eagle version="9.4.2">
 <drawing>
 <settings>
@@
 <label x="-27.94" y="162.56" size="1.778" layer="95"/>
 </segment>
+<segment>
+<pinref part="C_BAUX" gate="G$1" pin="OUT"/>
+<wire x1="-58.42" y1="149.86" x2="-48.26" y2="149.86" width="0.1524" layer="91"/>
+</segment>
 </net>
 <net name="25" class="0">
@@
 <junction x="-76.2" y="-5.08"/>
 <label x="-81.28" y="-2.54" size="1.778" layer="95"/>
-</segment>
-<segment>
-<pinref part="C_BAUX" gate="G$1" pin="OUT"/>
-<wire x1="-58.42" y1="149.86" x2="-48.26" y2="149.86" width="0.1524" layer="91"/>
 </segment>
 </net>
@@
 <segment>
 <pinref part="R19" gate="G$1" pin="2"/>
-<wire x1="41.91" y1="68.834" x2="41.91" y2="71.12" width="0.1524" layer="91"/>
 <wire x1="41.91" y1="71.12" x2="36.068" y2="71.12" width="0.1524" layer="91"/>
 <label x="36.068" y="73.406" size="1.778" layer="95"/>
+<pinref part="R20" gate="G$1" pin="1"/>
+<wire x1="41.91" y1="68.58" x2="41.91" y2="71.12" width="0.1524" layer="91"/>
+<junction x="41.91" y="71.12"/>
 </segment>
 <segment>
@@
 <segment>
 <pinref part="R21" gate="G$1" pin="1"/>
+<wire x1="69.85" y1="71.12" x2="59.69" y2="71.12" width="0.1524" layer="91"/>
+<label x="59.69" y="72.39" size="1.778" layer="95"/>
 <pinref part="R22" gate="G$1" pin="2"/>
 <wire x1="69.85" y1="68.58" x2="69.85" y2="71.12" width="0.1524" layer="91"/>
 <junction x="69.85" y="71.12"/>
-<wire x1="69.85" y1="71.12" x2="59.69" y2="71.12" width="0.1524" layer="91"/>
-<label x="59.69" y="72.39" size="1.778" layer="95"/>
-</segment>
-<segment>
+</segment>
+<segment>

Commit message: Adicao de Rotas e mudanca de nomes
Parts:
- renumbered SHUNTS to BORNE_SHUNTS
Changed lines of the file:
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@@
 <part name="BB_BE_C" library="diy-modules" deviceset="CURRENT-SENSOR-ACS712" device=""/>
 <part name="C_BAUX" library="diy-modules" deviceset="CURRENT-SENSOR-ACS712" device=""/>
-<part name="SHUNTS" library="con-amp-quick" library_urn="urn:adsk.eagle:library:125" deviceset="M02" device="" package3d_urn="urn:adsk.eagle:package:5956/1"/>
+<part name="BORNE_SHUNTS" library="con-amp-quick" library_urn="urn:adsk.eagle:library:125" deviceset="M02" device="" package3d_urn="urn:adsk.eagle:package:5956/1"/>
 </parts>
 <sheets>
@@
 <attribute name="VALUE" x="-88.9" y="160.02" size="1.778" layer="96"/>
 </instance>
-<instance part="SHUNTS" gate="G$1" x="-86.36" y="169.164" smashed="yes">
+<instance part="BORNE_SHUNTS" gate="G$1" x="-86.36" y="169.164" smashed="yes">
 <attribute name="VALUE" x="-88.9" y="164.084" size="1.778" layer="96"/>
 <attribute name="NAME" x="-88.9" y="175.006" size="1.778" layer="95"/>
@@
 </segment>
 <segment>
-<pinref part="SHUNTS" gate="G$1" pin="1"/>
+<pinref part="BORNE_SHUNTS" gate="G$1" pin="1"/>
 <wire x1="-78.74" y1="169.164" x2="-66.04" y2="169.164" width="0.1524" layer="91"/>
 <label x="-68.58" y="169.164" size="1.778" layer="95" align="bottom-right"/>
@@
 </segment>
 <segment>
-<pinref part="SHUNTS" gate="G$1" pin="2"/>
+<pinref part="BORNE_SHUNTS" gate="G$1" pin="2"/>
 <wire x1="-78.74" y1="171.704" x2="-66.04" y2="171.704" width="0.1524" layer="91"/>
 <label x="-68.58" y="171.704" size="1.778" layer="95" align="bottom-right"/>

Commit message: Limpeza e mudanca dos nomes
Update de organizacao
Parts:
- removed BB_BE_C: CURRENT-SENSOR-ACS712, diy-modules:CURRENT-SENSOR-ACS712
- removed BORNE_SHUNTS: (no value), con-amp-quick:M02
- removed TBEAM_LEFT, TBEAM_RIGHT: 61301311121, Headers:61301311121
- added 12-5: DC-DC-STEP-DOWN-LM2596, diy-modules:DC-DC-STEP-DOWN-LM2596
- added C_BP: CURRENT-SENSOR-ACS712, diy-modules:CURRENT-SENSOR-ACS712
- added R25, R27: 2.2k, rcl:R-EU_0204/7
- added R26, R28: 3.9k, rcl:R-EU_0204/7
- added SHUNTS, SL7, SUPPLY, TEMP1, TEMP2: (no value), con-amp-quick:M02
- added SL4: (no value), con-amp-quick:M03
- added U$1: TTGOBEAM, bibliotecattgo:TTGOBEAM
- SL2: device con-amp-quick:M05 -> con-amp-quick:M03
- SL3: device con-amp-quick:M05 -> con-amp-quick:M02
Connections:
- removed net EN: HC4067.EN
- removed net S0: HC4067.S0
- removed net S1: HC4067.S1
- removed net S2: HC4067.S2
- removed net S3: HC4067.S3
- removed net SIG: HC4067.SIG
- new net GND1: U$1.GND1
- new net GND2: U$1.GND2
- new net N$1: C_BP.OUT, R25.2
- new net N$2: C_BAUX.OUT, R27.2
- new net VI: 12-5.IN+, SUPPLY.2
- net 0: now also HC4067.S3, U$1.0; no longer TBEAM_RIGHT.5
- net 13: now also U$1.13; no longer R23.2, R24.1, TBEAM_LEFT.4
- net 14: now also U$1.14; no longer R13.1, R14.2, TBEAM_LEFT.5
- net 2: now also U$1.2; no longer R11.2, R12.1, TBEAM_LEFT.3
- net 21: now also SHUNTS.1, TEMP1.2, TEMP2.2, U$1.21; no longer BORNE_SHUNTS.2, TBEAM_RIGHT.10
- net 22: now also SHUNTS.2, TEMP1.1, TEMP2.1, U$1.22; no longer BORNE_SHUNTS.1, TBEAM_RIGHT.9
- net 23: now also U$1.23; no longer TBEAM_RIGHT.3
- net 25: now also U$1.25; no longer R1.1, R2.2, TBEAM_LEFT.6
- net 3.3V: now also U$1.3.3V; no longer TBEAM_RIGHT.11
- net 32: now also HC4067.S0, U$1.32; no longer TBEAM_LEFT.8
- net 33: now also HC4067.EN, U$1.33; no longer C_BAUX.OUT, TBEAM_LEFT.7
- net 34: now also HC4067.S2, U$1.34; no longer TBEAM_LEFT.10
- net 35: now also HC4067.S1, U$1.35; no longer TBEAM_LEFT.9
- net 3V3: now also HC4067.VCC, U$1.3V3; no longer TBEAM_RIGHT.7
- net 4: now also HC4067.SIG, U$1.4; no longer TBEAM_RIGHT.4
- net 5V: now also U$1.5V; no longer TBEAM_LEFT.1
- net BAT_AUX: now also R21.2, SL3.1; no longer R23.1, SL2.5
- net BB_IN: now also SL4.2; no longer SL2.4
- net BE_IN: now also SL4.1; no longer SL2.3
- net BTN_CRUZEIRO: now also SL7.2; no longer SL3.5
- net BTN_RE: now also SL2.3; no longer SL3.3
- net C0: now also R10.2, R9.1; no longer R3.2, R4.1
- net C1: now also R7.2, R8.1; no longer R5.1, R6.2
- net C10: now also R21.1, R22.2
- net C11: now also R1.1, R2.2
- net C12: now also R13.1, R14.2
- net C13: now also R27.1, R28.1
- net C2: now also R5.1, R6.2; no longer R7.2, R8.1
- net C3: now also R3.2, R4.1; no longer R10.2, R9.1
- net C4: now also R11.2, R12.1; no longer R21.1, R22.2
- net C5: now also R23.2, R24.1; no longer R19.2, R20.1
- net C6: now also R15.2, R16.1; no longer R17.1, R18.2
- net C7: now also R17.1, R18.2; no longer R15.2, R16.1
- net C8: now also R19.2, R20.1
- net C9: now also R25.1, R26.1
- net COOLER_D: now also SL3.2; no longer SL2.2
- net COOLER_E: now also R23.1, SL4.3; no longer R21.2, SL2.1
- net DMS_IN: now also SL2.2; no longer SL3.2
- net GND: now also 12-5.IN-, 12-5.OUT-, C_BP.GND, R26.2, R28.2, SUPPLY.1, U$1.GND; no longer TBEAM_LEFT.2, TBEAM_RIGHT.6, TBEAM_RIGHT.8
- net LORA1: now also U$1.LORA1; no longer TBEAM_RIGHT.13
- net LORA2: now also U$1.LORA2; no longer TBEAM_RIGHT.12
- net ON-OFF_MOTOR: now also SL7.1; no longer SL3.4
- net POT_IN: now also SL2.1; no longer SL3.1
- net RST: now also U$1.RST; no longer TBEAM_LEFT.11
- net RX: now also U$1.RX; no longer TBEAM_RIGHT.2
- net TX: now also U$1.TX; no longer TBEAM_RIGHT.1
- net VCC: now also 12-5.OUT+, C_BP.VCC; no longer HC4067.VCC
- net VN: now also U$1.VN; no longer TBEAM_LEFT.12
- net VP: now also U$1.VP; no longer TBEAM_LEFT.13
Other:
- moved on the sheet: C_BAUX, HC4067, R1, R11, R12, R13, R14, R15, R16, R17, R18, R19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
