File: latest/electric_project/hardware/PCB_WIDE_TRAILS/pcb_telemetria.brd (EAGLE design)
At the start: 160 x 75.9 mm, 48 parts

Commit message: att pra caqui baixar
ice crackerr
Parts:
- moved R27 1.27 mm to (150.5, 29.8)
- moved R28 1.27 mm to (150.5, 19.7)
- moved R7 1.27 mm to (156.8, 29.8)
- moved R8 1.27 mm to (156.8, 19.7)
- moved R19 0.63 mm to (14.6, 56.5)
- moved R20 0.63 mm to (14.6, 46.4)
Routing:
- net GND: track 5.34 -> 101.9 mm
- net 3V3: track 78.2 -> 83.7 mm
- net TX: track 93.6 -> 97.8 mm
- net RX: track 81.7 -> 84.8 mm
- net 33: track 99.0 -> 102.0 mm
- net 23: track 78.1 -> 81.0 mm
- net 21: track 129.3 -> 126.7 mm
- net C11: track 29.1 -> 31.5 mm
- net C15: track 197.0 -> 199.3 mm
- net C13: track 32.7 -> 34.8 mm
- net C14: track 213.7 -> 215.7 mm
- net C9: track 27.5 -> 29.3 mm
- net EXTRA1: track 14.8 -> 16.5 mm
- net C3: track 24.5 -> 26.1 mm
- net C10: track 28.3 -> 29.9 mm
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Other:
- board size 160 x 75.9 mm -> 159.4 x 75.9 mm

Commit message: veja agora ice
Routing:
- net GND: track 101.9 -> 100.7 mm
- removed copper zone on layer 1, net GND
Changed lines of the file:
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@@
 <grid distance="25" unitdist="mil" unit="mil" style="lines" multiple="1" display="no" altdistance="5" altunitdist="mil" altunit="mil"/>
 <layers>
-<layer number="1" name="Top" color="4" fill="1" visible="no" active="yes"/>
+<layer number="1" name="Top" color="4" fill="1" visible="yes" active="yes"/>
 <layer number="2" name="Route2" color="16" fill="1" visible="no" active="no"/>
 <layer number="3" name="Route3" color="17" fill="1" visible="no" active="no"/>
@@
 <contactref element="C3" pad="-"/>
 <contactref element="C5" pad="-"/>
-<polygon width="0.508" layer="1">
-<vertex x="-3.81" y="81.28"/>
-<vertex x="-3.81" y="-5.08"/>
-<vertex x="-1.27" y="-7.62"/>
-<vertex x="158.115" y="-7.62"/>
-<vertex x="164.465" y="-1.27"/>
-<vertex x="164.465" y="85.725"/>
-<vertex x="163.83" y="86.36"/>
-<vertex x="1.27" y="86.36"/>
-</polygon>
 <wire x1="16.51" y1="8.255" x2="15.875" y2="8.89" width="0.8128" layer="16"/>
 <wire x1="15.875" y1="13.335" x2="15.875" y2="8.89" width="0.8128" layer="16"/>
@@
 <wire x1="68.58" y1="69.85" x2="72.39" y2="69.85" width="0.8128" layer="16"/>
 <wire x1="80.645" y1="61.595" x2="80.645" y2="53.34" width="0.8128" layer="16"/>
-<wire x1="80.645" y1="53.34" x2="74.93" y2="47.625" width="0.8128" layer="16"/>
-<wire x1="74.93" y1="47.625" x2="73.025" y2="47.625" width="0.8128" layer="16"/>
-<wire x1="73.025" y1="47.625" x2="71.882" y2="46.482" width="0.8128" layer="16"/>
-<wire x1="71.882" y1="46.482" x2="71.882" y2="40.64" width="0.8128" layer="16"/>
+<wire x1="80.645" y1="53.34" x2="71.882" y2="44.577" width="0.8128" layer="16"/>
+<wire x1="71.882" y1="44.577" x2="71.882" y2="40.64" width="0.8128" layer="16"/>
 <wire x1="72.39" y1="69.85" x2="80.645" y2="61.595" width="0.8128" layer="16"/>
 <wire x1="123.19" y1="46.99" x2="128.27" y2="46.99" width="0.8128" layer="16"/>
