File: electric_project/Painel_barco/placa_painel.sch (EAGLE design)
At the start: 0 parts

Commit message: plaquinha extra pro painel
Parts:
- added X1: (no value), con-molex-micro-fit-3_0:HEADER_POS12_43045-1212
Connections:
- new net 21: X1.4
- new net 22: X1.6
- new net BB_IN: X1.12
- new net BE_IN: X1.1
- new net BTN_CRUZ: X1.10
- new net BTN_M: X1.9
- new net BTN_RE: X1.8
- new net DMS_IN: X1.7
- new net EXTRA2: X1.2
- new net N$1: X1.5
- new net N$2: X1.3
- new net POT_IN: X1.11
Other:
- note added: "MEASURE AND CONNECTORS"
- note added: "Panel Connectors"
