File: electric_project/Painel_barco/placa_painel.sch (EAGLE design)
At the start: 1 part

Commit message: placa_painel
Parts:
- added X2: (no value), con-molex-micro-fit-3_0:HEADER_POS10_43045-1012
- added X3: (no value), con-molex-micro-fit-3_0:HEADER_POS2_43045-0212
- added X4: (no value), con-ptr500:AK500/2
- added X5: (no value), con-ptr500:AK500/3
Connections:
- new net 1: X2.1
- new net 10: X2.10
- new net 2: X2.2
- new net 3: X2.3
- new net 4: X2.4
- new net 5: X2.5
- new net 6: X2.6
- new net 7: X2.7
- new net 8: X2.8
- new net 9: X2.9
- new net GND: X3.2
- new net VCC_12: X3.1
Other:
- note added: "12V Connector"
- note added: "CONNECTION BOARD"
- note added: "Motor Connectors"
- note added: "Telemetry Connectors"
- note removed: "MEASURE AND CONNECTORS"
- note removed: "Panel Connectors"
Changed lines of the file:
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@@
 <parts>
 <part name="X1" library="con-molex-micro-fit-3_0" deviceset="HEADER_POS12_?" device="43045-1212" override_package3d_urn="urn:adsk.eagle:package:15245313/2" override_package_urn="urn:adsk.eagle:footprint:15245314/1"/>
+<part name="X2" library="con-molex-micro-fit-3_0" deviceset="HEADER_POS10_?" device="43045-1012"/>
+<part name="X3" library="con-molex-micro-fit-3_0" deviceset="HEADER_POS2_?" device="43045-0212"/>
+<part name="X4" library="con-ptr500" library_urn="urn:adsk.eagle:library:181" deviceset="AK500/2" device="" package3d_urn="urn:adsk.eagle:package:9880/1"/>
+<part name="X5" library="con-ptr500" library_urn="urn:adsk.eagle:library:181" deviceset="AK500/3" device="" package3d_urn="urn:adsk.eagle:package:9883/1"/>
 </parts>
 <sheets>
@@
 <plain>
 <frame x1="-144.78" y1="45.72" x2="109.22" y2="195.58" columns="8" rows="5" layer="94"/>
-<text x="-17.78" y="185.42" size="5.08" layer="94" align="center">MEASURE AND CONNECTORS</text>
-<frame x1="-3.81" y1="111.76" x2="36.83" y2="162.56" columns="0" rows="0" layer="98" border-left="no" border-top="no" border-right="no" border-bottom="no"/>
+<text x="-17.78" y="180.34" size="5.08" layer="94" align="center">CONNECTION BOARD</text>
+<frame x1="-3.81" y1="121.92" x2="36.83" y2="162.56" columns="0" rows="0" layer="98" border-left="no" border-top="no" border-right="no" border-bottom="no"/>
 <frame x1="-130.048" y1="83.82" x2="-60.198" y2="162.56" columns="0" rows="0" layer="98" border-left="no" border-top="no" border-right="no" border-bottom="no"/>
-<text x="2.54" y="157.48" size="2.54" layer="94">Panel Connectors</text>
+<text x="0" y="157.48" size="2.54" layer="94">Telemetry Connectors</text>
+<frame x1="41.91" y1="121.92" x2="82.55" y2="162.56" columns="0" rows="0" layer="98" border-left="no" border-top="no" border-right="no" border-bottom="no"/>
+<text x="48.768" y="157.48" size="2.54" layer="94">Motor Connectors</text>
+<frame x1="-49.53" y1="121.92" x2="-8.89" y2="162.56" columns="0" rows="0" layer="98" border-left="no" border-top="no" border-right="no" border-bottom="no"/>
+<text x="-40.64" y="157.48" size="2.54" layer="94">12V Connector</text>
 </plain>
 <instances>
@@
 <attribute name="NAME" x="-1.016" y="146.558" size="1.778" layer="95" rot="R90"/>
 </instance>
+<instance part="X2" gate="G$1" x="63.5" y="147.32" smashed="yes" rot="R90">
+<attribute name="VALUE" x="78.74" y="146.05" size="1.778" layer="96" rot="R90"/>
+<attribute name="NAME" x="47.498" y="146.05" size="1.778" layer="95" rot="R90"/>
+</instance>
+<instance part="X3" gate="G$1" x="-27.94" y="147.32" smashed="yes" rot="R90">
+<attribute name="VALUE" x="-22.86" y="146.05" size="1.778" layer="96" rot="R90"/>
+<attribute name="NAME" x="-33.782" y="146.05" size="1.778" layer="95" rot="R90"/>
+</instance>
+<instance part="X4" gate="-1" x="-68.58" y="119.38" smashed="yes" rot="R270">
+<attribute name="NAME" x="-67.691" y="120.65" size="1.778" layer="95" rot="R90"/>
+</instance>
+<instance part="X4" gate="-2" x="-73.66" y="119.38" smashed="yes" rot="R270">
+<attribute name="NAME" x="-72.771" y="120.65" size="1.778" layer="95" rot="R90"/>
+<attribute name="VALUE" x="-77.343" y="123.19" size="1.778" layer="96" rot="R270"/>
+</instance>
+<instance part="X5" gate="-1" x="-83.82" y="119.38" smashed="yes" rot="R270">
+<attribute name="NAME" x="-82.931" y="120.65" size="1.778" layer="95" rot="R90"/>
+</instance>
+<instance part="X5" gate="-2" x="-88.9" y="119.38" smashed="yes" rot="R270">
+<attribute name="NAME" x="-88.011" y="120.65" size="1.778" layer="95" rot="R90"/>
+</instance>
+<instance part="X5" gate="-3" x="-93.98" y="119.38" smashed="yes" rot="R270">
+<attribute name="NAME" x="-93.091" y="120.65" size="1.778" layer="95" rot="R90"/>
+<attribute name="VALUE" x="-97.663" y="123.19" size="1.778" layer="96" rot="R270"/>
+</instance>
 </instances>
 <busses>
@@
 <wire x1="7.366" y1="142.748" x2="7.366" y2="127" width="0.1524" layer="91"/>
 <label x="7.366" y="127.508" size="1.778" layer="95" rot="R90"/>
+</segment>
+</net>
+<net name="1" class="0">
+<segment>
+<pinref part="X2" gate="G$1" pin="1"/>
+<wire x1="50.8" y1="142.24" x2="50.8" y2="134.62" width="0.1524" layer="91"/>
+<label x="50.8" y="137.16" size="1.778" layer="95" rot="R90"/>
+</segment>
+</net>
+<net name="2" class="0">
+<segment>
+<pinref part="X2" gate="G$1" pin="2"/>
+<wire x1="53.34" y1="142.24" x2="53.34" y2="134.62" width="0.1524" layer="91"/>
+<label x="53.34" y="137.16" size="1.778" layer="95" rot="R90"/>
+</segment>
+</net>
+<net name="3" class="0">
+<segment>
+<pinref part="X2" gate="G$1" pin="3"/>
+<wire x1="55.88" y1="142.24" x2="55.88" y2="134.62" width="0.1524" layer="91"/>
+<label x="55.88" y="137.16" size="1.778" layer="95" rot="R90"/>
+</segment>
+</net>
+<net name="4" class="0">
+<segment>
+<pinref part="X2" gate="G$1" pin="4"/>
+<wire x1="58.42" y1="142.24" x2="58.42" y2="134.62" width="0.1524" layer="91"/>
+<label x="58.42" y="137.16" size="1.778" layer="95" rot="R90"/>
+</segment>
+</net>
+<net name="5" class="0">
+<segment>
+<pinref part="X2" gate="G$1" pin="5"/>
+<wire x1="60.96" y1="142.24" x2="60.96" y2="134.62" width="0.1524" layer="91"/>
+<label x="60.96" y="137.16" size="1.778" layer="95" rot="R90"/>
+</segment>
+</net>
+<net name="6" class="0">
+<segment>
+<pinref part="X2" gate="G$1" pin="6"/>
+<wire x1="63.5" y1="142.24" x2="63.5" y2="134.62" width="0.1524" layer="91"/>
+<label x="63.5" y="137.16" size="1.778" layer="95" rot="R90"/>
+</segment>
+</net>
+<net name="7" class="0">
+<segment>
+<pinref part="X2" gate="G$1" pin="7"/>
+<wire x1="66.04" y1="142.24" x2="66.04" y2="134.62" width="0.1524" layer="91"/>
+<label x="66.04" y="137.16" size="1.778" layer="95" rot="R90"/>
+</segment>
+</net>
+<net name="8" class="0">
+<segment>
+<pinref part="X2" gate="G$1" pin="8"/>
+<wire x1="68.58" y1="142.24" x2="68.58" y2="134.62" width="0.1524" layer="91"/>
+<label x="68.58" y="137.16" size="1.778" layer="95" rot="R90"/>
+</segment>
+</net>
+<net name="9" class="0">
+<segment>
+<pinref part="X2" gate="G$1" pin="9"/>
+<wire x1="71.12" y1="142.24" x2="71.12" y2="134.62" width="0.1524" layer="91"/>
+<label x="71.12" y="137.16" size="1.778" layer="95" rot="R90"/>
+</segment>
+</net>
+<net name="10" class="0">
+<segment>
+<pinref part="X2" gate="G$1" pin="10"/>
+<wire x1="73.66" y1="142.24" x2="73.66" y2="134.62" width="0.1524" layer="91"/>
+<label x="73.66" y="137.16" size="1.778" layer="95" rot="R90"/>
+</segment>
+</net>
+<net name="VCC_12" class="0">
+<segment>
+<pinref part="X3" gate="G$1" pin="1"/>
+<wire x1="-30.48" y1="142.24" x2="-30.48" y2="129.54" width="0.1524" layer="91"/>
+<label x="-30.48" y="129.54" size="1.778" layer="95" rot="R180" xref="yes"/>
+</segment>
+</net>
+<net name="GND" class="0">
+<segment>
+<pinref part="X3" gate="G$1" pin="2"/>
+<wire x1="-27.94" y1="142.24" x2="-27.94" y2="129.54" width="0.1524" layer="91"/>
+<label x="-27.94" y="129.54" size="1.778" layer="95" xref="yes"/>
 </segment>
 </net>
@@
 </drawing>
 <compatibility>
+<note version="8.2" severity="warning">
+Since Version 8.2, EAGLE supports online libraries. The ids
+of those online libraries will not be understood (or retained)
+with this version.
+</note>
+<note version="8.3" severity="warning">
+Since Version 8.3, EAGLE supports URNs for individual library
+assets (packages, symbols, and devices). The URNs of those assets
+will not be understood (or retained) with this version.
+</note>
 <note version="8.3" severity="warning">
 Since Version 8.3, EAGLE supports the association of 3D packages

Commit message: update
Connections:
- net 1 renamed RED_ONOFF_45V_PH
- removed net 10: X2.10
- removed net 2: X2.2
- removed net 3: X2.3
- removed net 4: X2.4
- removed net 5: X2.5
- removed net 6: X2.6
- removed net 7: X2.7
- removed net 8: X2.8
- removed net 9: X2.9
- removed net BTN_CRUZ: X1.10
- removed net BTN_M: X1.9
- removed net POT_IN: X1.11
- new net BLACK_GND: X2.4, X2.5, X5-3.KL
- new net BLUE_5V: X2.2, X5-1.KL
- new net N$6: X4-1.KL
- new net N$7: X4-2.KL
- new net PURP_45V_ONOFF_BACK: X1.9, X2.7
- new net WHITE_CRUISE: X1.10, X2.6
- new net YEL_POT_MEASURE: X1.11, X2.3, X5-2.KL
- net GND: now also X2.10, X2.8, X2.9
Other:
- note added: "CONNECTIONS"
- note removed: "CONNECTION BOARD"
- moved on the sheet: X4-1, X4-2, X5-1, X5-2, X5-3
