File: electric_project/Painel_barco/placa_painel.sch (EAGLE design)
At the start: 15 parts, among them IC1 7805TV

Commit message: up
Parts:
- removed R3, R4: (no value), rcl:R-EU_0204/7
- added BB, BE: (no value), con-ptr500:AK500/3
- added BB_IN, BE_IN, DMS: (no value), con-ptr500:AK500/2
- renumbered X1 to TELE_CON, X2 to MOTOR_CON
Connections:
- removed net BB_IN: TELE_CON.12
- removed net BE_IN: TELE_CON.1
- removed net DMS_IN: TELE_CON.7
- removed net N$8: R3.1, R4.2
- new net BB_AUTO: BB-1.KL, BB_IN-2.KL
- new net BB_RET: BB-2.KL, BB_IN-1.KL, TELE_CON.12
- new net BE_AUTO: BE-1.KL, BE_IN-2.KL
- new net BE_RET: BE-2.KL, BE_IN-1.KL, TELE_CON.1
- new net WHITE_DMS: DMS-2.KL, MOTOR_CON.1, TELE_CON.7
- net 21: now also X7.4; no longer X7.3
- net 22: now also X7.2; no longer X7.4
- net GND: now also DMS-1.KL; no longer R4.1
- net PURP_45V_ONOFF_BACK: no longer R3.2
- net VCC_12: now also BB-3.KL, BE-3.KL
- net VCC_5V: now also X7.3; no longer X7.2
- net WHITE_CRUISE: no longer MOTOR_CON.1
Other:
- note added: "BB"
- note added: "BE"
- note added: "DMS"
- moved on the sheet: ON_OFF-1, ON_OFF-2, POT-1, POT-2, POT-3, R1, R2, REV-1, REV-2
