File: electric_project/Painel_barco/placa_painel.brd (EAGLE design)
At the start: 160 x 100 mm, 1 part

Commit message: placa_painel
Parts:
- added X2: (no value), con-molex-micro-fit-3_0:43045-1012
- added X3: (no value), con-molex-micro-fit-3_0:43045-0212
- added X4: (no value), con-ptr500:AK500/2
- added X5: (no value), con-ptr500:AK500/3
- moved X1 72.3 mm to (5.08, 14.0), turned to 270 degrees
Connections:
- new net 1: X2.P$1
- new net 10: X2.P$10
- new net 2: X2.P$2
- new net 3: X2.P$3
- new net 4: X2.P$4
- new net 5: X2.P$5
- new net 6: X2.P$6
- new net 7: X2.P$7
- new net 8: X2.P$8
- new net 9: X2.P$9
- new net GND: X3.P$2
- new net VCC_12: X3.P$1
Routing:
- net N$3: track 0.00 -> 11.4 mm
Other:
- board size 160 x 100 mm -> 49.8 x 63.3 mm
Changed lines of the file:
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@@
 <board>
 <plain>
-<wire x1="0" y1="0" x2="160" y2="0" width="0" layer="20"/>
-<wire x1="160" y1="0" x2="160" y2="100" width="0" layer="20"/>
-<wire x1="160" y1="100" x2="0" y2="100" width="0" layer="20"/>
-<wire x1="0" y1="100" x2="0" y2="0" width="0" layer="20"/>
+<wire x1="0" y1="0" x2="49.764" y2="-0.127" width="0" layer="20"/>
+<wire x1="49.764" y1="-0.127" x2="49.764" y2="63.043" width="0" layer="20"/>
+<wire x1="49.764" y1="63.043" x2="0" y2="63.17" width="0" layer="20"/>
+<wire x1="0" y1="63.17" x2="0" y2="0" width="0" layer="20"/>
 </plain>
 <attributes>
@@
 </autorouter>
 <elements>
-<element name="X1" library="con-molex-micro-fit-3_0" package="43045-1212" override_package3d_urn="urn:adsk.eagle:package:15245313/2" override_package_urn="urn:adsk.eagle:footprint:15245314/1" value="" x="67.31" y="50.8" smashed="yes"/>
+<element name="X1" library="con-molex-micro-fit-3_0" package="43045-1212" override_package3d_urn="urn:adsk.eagle:package:15245313/2" override_package_urn="urn:adsk.eagle:footprint:15245314/1" value="" x="5.08" y="13.97" smashed="yes" rot="R270"/>
+<element name="X2" library="con-molex-micro-fit-3_0" package="43045-1012" value="" x="5.08" y="38.1" smashed="yes" rot="R270"/>
+<element name="X3" library="con-molex-micro-fit-3_0" package="43045-0212" value="" x="5.08" y="54.61" smashed="yes" rot="R270"/>
+<element name="X4" library="con-ptr500" library_urn="urn:adsk.eagle:library:181" package="AK500/2" package3d_urn="urn:adsk.eagle:package:9880/1" value="" x="-6.35" y="6.35" smashed="yes">
+<attribute name="MF" value="" x="-6.35" y="6.35" size="1.778" layer="27" display="off"/>
+<attribute name="MPN" value="" x="-6.35" y="6.35" size="1.778" layer="27" display="off"/>
+<attribute name="NAME" x="-11.43" y="10.795" size="1.778" layer="25" ratio="10"/>
+<attribute name="OC_FARNELL" value="unknown" x="-6.35" y="6.35" size="1.778" layer="27" display="off"/>
+<attribute name="OC_NEWARK" value="unknown" x="-6.35" y="6.35" size="1.778" layer="27" display="off"/>
+<attribute name="VALUE" x="-11.43" y="0.635" size="1.778" layer="27" ratio="10"/>
+</element>
+<element name="X5" library="con-ptr500" library_urn="urn:adsk.eagle:library:181" package="AK500/3" package3d_urn="urn:adsk.eagle:package:9883/1" value="" x="-3.81" y="-7.62" smashed="yes">
+<attribute name="MF" value="" x="-3.81" y="-7.62" size="1.778" layer="27" display="off"/>
+<attribute name="MPN" value="" x="-3.81" y="-7.62" size="1.778" layer="27" display="off"/>
+<attribute name="NAME" x="-11.4046" y="-3.175" size="1.778" layer="25" ratio="10"/>
+<attribute name="OC_FARNELL" value="unknown" x="-3.81" y="-7.62" size="1.778" layer="27" display="off"/>
+<attribute name="OC_NEWARK" value="unknown" x="-3.81" y="-7.62" size="1.778" layer="27" display="off"/>
+<attribute name="VALUE" x="-11.4046" y="-13.335" size="1.778" layer="27" ratio="10"/>
+</element>
 </elements>
 <signals>
@@
 <signal name="N$2">
 <contactref element="X1" pad="P$3"/>
+</signal>
+<signal name="1">
+<contactref element="X2" pad="P$1"/>
+</signal>
+<signal name="2">
+<contactref element="X2" pad="P$2"/>
+</signal>
+<signal name="3">
+<contactref element="X2" pad="P$3"/>
+</signal>
+<signal name="4">
+<contactref element="X2" pad="P$4"/>
+</signal>
+<signal name="5">
+<contactref element="X2" pad="P$5"/>
+</signal>
+<signal name="6">
+<contactref element="X2" pad="P$6"/>
+</signal>
+<signal name="7">
+<contactref element="X2" pad="P$7"/>
+</signal>
+<signal name="8">
+<contactref element="X2" pad="P$8"/>
+</signal>
+<signal name="9">
+<contactref element="X2" pad="P$9"/>
+</signal>
+<signal name="10">
+<contactref element="X2" pad="P$10"/>
+</signal>
+<signal name="N$3">
+<wire x1="22.479" y1="33.528" x2="11.049" y2="33.528" width="0.1524" layer="1"/>
+</signal>
+<signal name="VCC_12">
+<contactref element="X3" pad="P$1"/>
+</signal>
+<signal name="GND">
+<contactref element="X3" pad="P$2"/>
 </signal>
 </signals>
@@
 </drawing>
 <compatibility>
+<note version="8.2" severity="warning">
+Since Version 8.2, EAGLE supports online libraries. The ids
+of those online libraries will not be understood (or retained)
+with this version.
+</note>
+<note version="8.3" severity="warning">
+Since Version 8.3, EAGLE supports URNs for individual library
+assets (packages, symbols, and devices). The URNs of those assets
+will not be understood (or retained) with this version.
+</note>
 <note version="8.3" severity="warning">
 Since Version 8.3, EAGLE supports the association of 3D packages

Commit message: update
Parts:
- moved X5 77.2 mm to (43.8, 53.1), turned to 90 degrees
- moved X4 49.5 mm to (43.2, 7.62), turned to 90 degrees
Connections:
- net 1 renamed RED_ONOFF_45V_PH
- removed net 10: X2.P$10
- removed net 2: X2.P$2
- removed net 3: X2.P$3
- removed net 4: X2.P$4
- removed net 5: X2.P$5
- removed net 6: X2.P$6
- removed net 7: X2.P$7
- removed net 8: X2.P$8
- removed net 9: X2.P$9
- removed net BTN_CRUZ: X1.P$10
- removed net BTN_M: X1.P$9
- removed net POT_IN: X1.P$11
- new net BLACK_GND: X2.P$4, X2.P$5, X5.3
- new net BLUE_5V: X2.P$2, X5.1
- new net N$6: X4.1
- new net N$7: X4.2
- new net PURP_45V_ONOFF_BACK: X1.P$9, X2.P$7
- new net WHITE_CRUISE: X1.P$10, X2.P$6
- new net YEL_POT_MEASURE: X1.P$11, X2.P$3, X5.2
- net GND: now also X2.P$10, X2.P$8, X2.P$9
Routing:
- net N$3: track 11.4 -> 0.00 mm
Changed lines of the file:
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@@
 <element name="X2" library="con-molex-micro-fit-3_0" package="43045-1012" value="" x="5.08" y="38.1" smashed="yes" rot="R270"/>
 <element name="X3" library="con-molex-micro-fit-3_0" package="43045-0212" value="" x="5.08" y="54.61" smashed="yes" rot="R270"/>
-<element name="X4" library="con-ptr500" library_urn="urn:adsk.eagle:library:181" package="AK500/2" package3d_urn="urn:adsk.eagle:package:9880/1" value="" x="-6.35" y="6.35" smashed="yes">
-<attribute name="MF" value="" x="-6.35" y="6.35" size="1.778" layer="27" display="off"/>
-<attribute name="MPN" value="" x="-6.35" y="6.35" size="1.778" layer="27" display="off"/>
-<attribute name="NAME" x="-11.43" y="10.795" size="1.778" layer="25" ratio="10"/>
-<attribute name="OC_FARNELL" value="unknown" x="-6.35" y="6.35" size="1.778" layer="27" display="off"/>
-<attribute name="OC_NEWARK" value="unknown" x="-6.35" y="6.35" size="1.778" layer="27" display="off"/>
-<attribute name="VALUE" x="-11.43" y="0.635" size="1.778" layer="27" ratio="10"/>
+<element name="X4" library="con-ptr500" library_urn="urn:adsk.eagle:library:181" package="AK500/2" package3d_urn="urn:adsk.eagle:package:9880/1" value="" x="43.18" y="7.62" smashed="yes" rot="R90">
+<attribute name="MF" value="" x="43.18" y="7.62" size="1.778" layer="27" rot="R90" display="off"/>
+<attribute name="MPN" value="" x="43.18" y="7.62" size="1.778" layer="27" rot="R90" display="off"/>
+<attribute name="NAME" x="38.735" y="2.54" size="1.778" layer="25" ratio="10" rot="R90"/>
+<attribute name="OC_FARNELL" value="unknown" x="43.18" y="7.62" size="1.778" layer="27" rot="R90" display="off"/>
+<attribute name="OC_NEWARK" value="unknown" x="43.18" y="7.62" size="1.778" layer="27" rot="R90" display="off"/>
+<attribute name="VALUE" x="48.895" y="2.54" size="1.778" layer="27" ratio="10" rot="R90"/>
 </element>
-<element name="X5" library="con-ptr500" library_urn="urn:adsk.eagle:library:181" package="AK500/3" package3d_urn="urn:adsk.eagle:package:9883/1" value="" x="-3.81" y="-7.62" smashed="yes">
-<attribute name="MF" value="" x="-3.81" y="-7.62" size="1.778" layer="27" display="off"/>
-<attribute name="MPN" value="" x="-3.81" y="-7.62" size="1.778" layer="27" display="off"/>
-<attribute name="NAME" x="-11.4046" y="-3.175" size="1.778" layer="25" ratio="10"/>
-<attribute name="OC_FARNELL" value="unknown" x="-3.81" y="-7.62" size="1.778" layer="27" display="off"/>
-<attribute name="OC_NEWARK" value="unknown" x="-3.81" y="-7.62" size="1.778" layer="27" display="off"/>
-<attribute name="VALUE" x="-11.4046" y="-13.335" size="1.778" layer="27" ratio="10"/>
+<element name="X5" library="con-ptr500" library_urn="urn:adsk.eagle:library:181" package="AK500/3" package3d_urn="urn:adsk.eagle:package:9883/1" value="" x="43.815" y="53.086" smashed="yes" rot="R90">
+<attribute name="MF" value="" x="43.815" y="53.086" size="1.778" layer="27" rot="R90" display="off"/>
+<attribute name="MPN" value="" x="43.815" y="53.086" size="1.778" layer="27" rot="R90" display="off"/>
+<attribute name="NAME" x="39.37" y="45.4914" size="1.778" layer="25" ratio="10" rot="R90"/>
+<attribute name="OC_FARNELL" value="unknown" x="43.815" y="53.086" size="1.778" layer="27" rot="R90" display="off"/>
+<attribute name="OC_NEWARK" value="unknown" x="43.815" y="53.086" size="1.778" layer="27" rot="R90" display="off"/>
+<attribute name="VALUE" x="49.53" y="45.4914" size="1.778" layer="27" ratio="10" rot="R90"/>
 </element>
 </elements>
@@
 <contactref element="X1" pad="P$8"/>
 </signal>
-<signal name="POT_IN">
-<contactref element="X1" pad="P$11"/>
-</signal>
 <signal name="BB_IN">
 <contactref element="X1" pad="P$12"/>
@@
 <signal name="BE_IN">
 <contactref element="X1" pad="P$1"/>
-</signal>
-<signal name="BTN_CRUZ">
-<contactref element="X1" pad="P$10"/>
-</signal>
-<signal name="BTN_M">
-<contactref element="X1" pad="P$9"/>
 </signal>
 <signal name="EXTRA2">
@@
 <contactref element="X1" pad="P$3"/>
 </signal>
-<signal name="1">
+<signal name="RED_ONOFF_45V_PH">
 <contactref element="X2" pad="P$1"/>
 </signal>
-<signal name="2">
+<signal name="BLUE_5V">
 <contactref element="X2" pad="P$2"/>
+<contactref element="X5" pad="1"/>
+<wire x1="5.08" y1="35.1" x2="43.815" y2="48.0822" width="0" layer="19" extent="1-1"/>
 </signal>
-<signal name="3">
+<signal name="YEL_POT_MEASURE">
 <contactref element="X2" pad="P$3"/>
+<contactref element="X1" pad="P$11"/>
+<contactref element="X5" pad="2"/>
+<wire x1="5.08" y1="38.1" x2="43.815" y2="53.086" width="0" layer="19" extent="1-1"/>
+<wire x1="8.08" y1="18.47" x2="5.08" y2="38.1" width="0" layer="19" extent="1-1"/>
 </signal>
-<signal name="4">
-<contactref element="X2" pad="P$4"/>
+<signal name="WHITE_CRUISE">
+<contactref element="X2" pad="P$6"/>
+<contactref element="X1" pad="P$10"/>
+<wire x1="8.08" y1="15.47" x2="8.08" y2="32.1" width="0" layer="19" extent="1-1"/>
 </signal>
-<signal name="5">
-<contactref element="X2" pad="P$5"/>
-</signal>
-<signal name="6">
-<contactref element="X2" pad="P$6"/>
-</signal>
-<signal name="7">
+<signal name="PURP_45V_ONOFF_BACK">
 <contactref element="X2" pad="P$7"/>
-</signal>
-<signal name="8">
-<contactref element="X2" pad="P$8"/>
-</signal>
-<signal name="9">
-<contactref element="X2" pad="P$9"/>
-</signal>
-<signal name="10">
-<contactref element="X2" pad="P$10"/>
-</signal>
-<signal name="N$3">
-<wire x1="22.479" y1="33.528" x2="11.049" y2="33.528" width="0.1524" layer="1"/>
+<contactref element="X1" pad="P$9"/>
+<wire x1="8.08" y1="12.47" x2="8.08" y2="35.1" width="0" layer="19" extent="1-1"/>
 </signal>
 <signal name="VCC_12">
@@
 <signal name="GND">
 <contactref element="X3" pad="P$2"/>
+<contactref element="X2" pad="P$8"/>
+<contactref element="X2" pad="P$9"/>
+<contactref element="X2" pad="P$10"/>
+<wire x1="8.08" y1="44.1" x2="8.08" y2="54.61" width="0" layer="19" extent="1-1"/>
+<wire x1="8.08" y1="41.1" x2="8.08" y2="44.1" width="0" layer="19" extent="1-1"/>
+<wire x1="8.08" y1="38.1" x2="8.08" y2="41.1" width="0" layer="19" extent="1-1"/>
+</signal>
+<signal name="BLACK_GND">
+<contactref element="X2" pad="P$4"/>
+<contactref element="X2" pad="P$5"/>
+<contactref element="X5" pad="3"/>
+<wire x1="5.08" y1="44.1" x2="43.815" y2="58.0898" width="0" layer="19" extent="1-1"/>
+<wire x1="5.08" y1="41.1" x2="5.08" y2="44.1" width="0" layer="19" extent="1-1"/>
+</signal>
+<signal name="N$6">
+<contactref element="X4" pad="1"/>
+</signal>
+<signal name="N$7">
+<contactref element="X4" pad="2"/>
 </signal>
 </signals>
