File: electric_project/Painel_barco/Placa_painel_Revisao.sch (EAGLE design)
At the start: 15 parts, among them IC1 7805TV

Commit message: up
Parts:
- removed R3, R4: (no value), rcl:R-EU_0204/7
- removed X1: (no value), con-molex-micro-fit-3_0:HEADER_POS12_43045-1212
- removed X2: (no value), con-molex-micro-fit-3_0:HEADER_POS10_43045-1012
- removed X3: (no value), con-molex-micro-fit-3_0:HEADER_POS2_43045-0212
- added BB, BE: (no value), con-ptr500:AK500/3
- added DMS, RADIO: (no value), con-ptr500:AK500/2
- added MOTOR_CON: (no value), con-molex-micro-fit-3_0:HEADER_POS10_43045-1012
- added TELE_CON: (no value), con-molex-micro-fit-3_0:HEADER_POS12_43045-1212
- added U$1: CON_HOLE, bibliotecattgo:CON_HOLE
Connections:
- removed net BB_IN: X1.12
- removed net BE_IN: X1.1
- removed net DMS_IN: X1.7
- removed net GND: C1.-, C2.-, IC1.GND, IC2.7, R2.1, R4.1, REV-1.KL, X2.4, X2.5, X3.1, X7.1
- removed net N$1: X1.5
- removed net N$2: X1.3
- removed net N$8: R3.1, R4.2
- new net BB_AUTO: BB-1.KL, U$1.P$6
- new net BB_RET: BB-2.KL, TELE_CON.12, U$1.P$2
- new net BE_AUTO: BE-1.KL, U$1.P$4
- new net BE_RET: BE-2.KL, TELE_CON.1, U$1.P$5
- new net WHITE_DMS: DMS-1.KL, MOTOR_CON.5, TELE_CON.7
- net 21: now also TELE_CON.3, TELE_CON.4, X7.4; no longer X1.4, X7.3
- net 22: now also TELE_CON.5, TELE_CON.6, X7.2; no longer X1.6, X7.4
- net BLACK_GND: now also C1.-, C2.-, DMS-2.KL, IC1.GND, IC2.7, MOTOR_CON.1, MOTOR_CON.2, MOTOR_CON.3, MOTOR_CON.6, R2.1, RADIO-1.KL, REV-1.KL, U$1.P$1, X7.1; no longer X2.10, X2.9
- net BLUE_5V: now also MOTOR_CON.9; no longer X2.7
- net BROWN_REVERSE: now also MOTOR_CON.4, TELE_CON.8; no longer X1.8, X2.3
- net EXTRA2: now also TELE_CON.2; no longer X1.2
- net ONOFF_MOTOR: now also TELE_CON.9; no longer X1.9
- net PURP_45V_ONOFF_BACK: now also MOTOR_CON.8; no longer R3.2, X2.2
- net RED_ONOFF_45V_PH: now also MOTOR_CON.7; no longer X2.6
- net VCC_12: now also BB-3.KL, BE-3.KL, RADIO-2.KL, U$1.P$3; no longer X3.2
- net VCC_5V: now also X7.3; no longer X7.2
- net WHITE_CRUISE: now also TELE_CON.10; no longer X1.10, X2.1
- net YEL_POT_MEASURE: now also MOTOR_CON.10, TELE_CON.11; no longer X1.11, X2.8
Other:
- note added: "BB"
- note added: "BE"
- note added: "DMS"
- note removed: "12V Connector"
- moved on the sheet: ON_OFF-1, ON_OFF-2, POT-1, POT-2, POT-3, R1, R2, REV-1, REV-2, X7
