File: electric_project/Painel_barco/Placa_painel_Revisao.brd (EAGLE design)
At the start: 100 x 70 mm, 17 parts, among them IC1 7805TV

Commit message: up
Routing:
- net BLACK_GND: track 305.8 -> 291.5 mm
- net WHITE_DMS: track 72.9 -> 86.6 mm
- net BB_RET: track 92.8 -> 84.9 mm
- net ONOFF_DOWN: track 45.8 -> 51.1 mm
- net YEL_POT_MEASURE: track 85.6 -> 87.1 mm
