File: electric_project/Painel_barco/trying/placa_painel.sch (EAGLE design)
At the start: 18 parts, among them IC1 7805TV

Commit message: up
Connections:
- net 21: now also X7.1; no longer X7.4
- net 22: now also X7.3; no longer X7.2
- net BLACK_GND: now also X7.2; no longer X7.1
- net BROWN_REVERSE: now also MOTOR_CON.2; no longer MOTOR_CON.1
- net VCC_5V: now also X7.4; no longer X7.3
- net WHITE_DMS: now also MOTOR_CON.1; no longer MOTOR_CON.2
