File: electric_project/hardware/PCB_WIDE_TRAILS/pcb_telemetria_wide.brd (EAGLE design)
At the start: 159.4 x 75.9 mm, 48 parts

Commit message: up
Routing:
- net VCC: track 57.3 -> 59.4 mm
Changed lines of the file:
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@@
 <drawing>
 <settings>
-<setting alwaysvectorfont="yes"/>
+<setting alwaysvectorfont="no"/>
 <setting verticaltext="up"/>
 </settings>
 <grid distance="25" unitdist="mil" unit="mil" style="lines" multiple="1" display="no" altdistance="5" altunitdist="mil" altunit="mil"/>
 <layers>
-<layer number="1" name="Top" color="4" fill="1" visible="no" active="yes"/>
+<layer number="1" name="Top" color="4" fill="1" visible="yes" active="yes"/>
 <layer number="2" name="Route2" color="16" fill="1" visible="no" active="no"/>
 <layer number="3" name="Route3" color="17" fill="1" visible="no" active="no"/>
@@
 <layer number="17" name="Pads" color="2" fill="1" visible="yes" active="yes"/>
 <layer number="18" name="Vias" color="2" fill="1" visible="yes" active="yes"/>
-<layer number="19" name="Unrouted" color="6" fill="1" visible="no" active="yes"/>
-<layer number="20" name="Dimension" color="24" fill="1" visible="no" active="yes"/>
+<layer number="19" name="Unrouted" color="6" fill="1" visible="yes" active="yes"/>
+<layer number="20" name="Dimension" color="24" fill="1" visible="yes" active="yes"/>
 <layer number="21" name="tPlace" color="7" fill="1" visible="yes" active="yes"/>
 <layer number="22" name="bPlace" color="7" fill="1" visible="no" active="yes"/>
-<layer number="23" name="tOrigins" color="15" fill="1" visible="no" active="yes"/>
-<layer number="24" name="bOrigins" color="15" fill="1" visible="no" active="yes"/>
-<layer number="25" name="tNames" color="7" fill="1" visible="no" active="yes"/>
-<layer number="26" name="bNames" color="7" fill="1" visible="no" active="yes"/>
+<layer number="23" name="tOrigins" color="15" fill="1" visible="yes" active="yes"/>
+<layer number="24" name="bOrigins" color="15" fill="1" visible="yes" active="yes"/>
+<layer number="25" name="tNames" color="7" fill="1" visible="yes" active="yes"/>
+<layer number="26" name="bNames" color="7" fill="1" visible="yes" active="yes"/>
 <layer number="27" name="tValues" color="7" fill="1" visible="yes" active="yes"/>
 <layer number="28" name="bValues" color="7" fill="1" visible="yes" active="yes"/>
@@
 <wire x1="128.27" y1="46.99" x2="128.905" y2="46.355" width="0.8128" layer="16"/>
 <wire x1="123.19" y1="65.405" x2="128.905" y2="65.405" width="0.8128" layer="16"/>
+<wire x1="128.27" y1="46.99" x2="128.905" y2="65.405" width="0" layer="19" extent="16-16"/>
+<wire x1="111.506" y1="40.64" x2="123.19" y2="46.99" width="0" layer="19" extent="1-1"/>
+<wire x1="80.645" y1="53.34" x2="111.506" y2="40.64" width="0" layer="19" extent="16-16"/>
+<wire x1="53.34" y1="42.545" x2="64.77" y2="42.545" width="0" layer="19" extent="1-1"/>
+<wire x1="49.53" y1="42.545" x2="53.34" y2="42.545" width="0" layer="19" extent="1-1"/>
+<wire x1="45.72" y1="42.545" x2="49.53" y2="42.545" width="0" layer="19" extent="1-1"/>
+<wire x1="41.275" y1="42.545" x2="45.72" y2="42.545" width="0" layer="19" extent="1-1"/>
+<wire x1="36.83" y1="42.545" x2="41.275" y2="42.545" width="0" layer="19" extent="1-1"/>
+<wire x1="33.02" y1="42.545" x2="36.83" y2="42.545" width="0" layer="19" extent="1-1"/>
+<wire x1="29.21" y1="42.545" x2="33.02" y2="42.545" width="0" layer="19" extent="1-1"/>
+<wire x1="26.035" y1="42.545" x2="29.21" y2="42.545" width="0" layer="19" extent="1-1"/>
+<wire x1="22.225" y1="42.545" x2="26.035" y2="42.545" width="0" layer="19" extent="1-1"/>
+<wire x1="18.288" y1="42.545" x2="22.225" y2="42.545" width="0" layer="19" extent="1-1"/>
+<wire x1="14.605" y1="42.545" x2="18.288" y2="42.545" width="0" layer="19" extent="1-1"/>
+<wire x1="10.795" y1="42.545" x2="14.605" y2="42.545" width="0" layer="19" extent="1-1"/>
+<wire x1="6.985" y1="42.545" x2="10.795" y2="42.545" width="0" layer="19" extent="1-1"/>
+<wire x1="3.175" y1="42.545" x2="6.985" y2="42.545" width="0" layer="19" extent="1-1"/>
+<wire x1="82.885" y1="7.32" x2="72.485" y2="32.22" width="0" layer="19" extent="1-1"/>
+<wire x1="20.955" y1="13.335" x2="22.225" y2="42.545" width="0" layer="19" extent="1-1"/>
+<wire x1="150.495" y1="15.875" x2="128.905" y2="46.355" width="0" layer="19" extent="1-1"/>
+<wire x1="156.845" y1="15.875" x2="150.495" y2="15.875" width="0" layer="19" extent="1-1"/>
 </signal>
 <signal name="22">
@@
 <contactref element="C3" pad="+"/>
 <wire x1="123.19" y1="60.325" x2="128.905" y2="60.325" width="0.508" layer="16"/>
-<wire x1="128.905" y1="60.325" x2="133.35" y2="55.88" width="1.016" layer="16"/>
-<wire x1="133.35" y1="41.91" x2="132.715" y2="41.275" width="1.016" layer="16"/>
+<wire x1="128.905" y1="60.325" x2="135.89" y2="53.34" width="1.016" layer="16"/>
+<wire x1="135.89" y1="44.45" x2="132.715" y2="41.275" width="1.016" layer="16"/>
 <wire x1="132.715" y1="41.275" x2="128.905" y2="41.275" width="1.016" layer="16"/>
-<wire x1="133.35" y1="55.88" x2="133.35" y2="41.91" width="1.016" layer="16"/>
+<wire x1="135.89" y1="53.34" x2="135.89" y2="44.45" width="1.016" layer="16"/>
 <wire x1="128.905" y1="41.275" x2="123.825" y2="41.275" width="1.016" layer="16"/>
 <wire x1="123.825" y1="41.275" x2="123.19" y2="41.91" width="1.016" layer="16"/>
